File: KiCAD/PrawnDO_Breakout_Connectorized_single_buffers.kicad_pcb (KiCad board)
At the start: 2 copper layers, 154.4 x 86.8 mm, 90 parts, among them J1 do15, J10 do6, J11 do5, J12 do4, J13 do3, J14 do2, J15 do1, J16 Ext. Trig., J17 Ext. Clk., J18 do0, J2 do14, J3 do13, J4 do11, J5 do12, J6 do10, J7 do9, J8 do8, J9 do7, U1 74LVC2G34DCKR, U11 74LVC1G34, U12 74LVC2G34DCKR, U13 74LVC2G34DCKR, U14 74LVC2G34DCKR, U15 74LVC2G34DCKR, U16 74LVC2G34DCKR, U17 74LVC2G34DCKR, U18 74LVC2G34DCKR, U19 74LVC2G34DCKR, U2 74LVC2G34DCKR, U2 Pico, U3 74LVC2G34DCKR, U4 74LVC2G34DCKR, U5 74LVC2G34DCKR, U6 74LVC2G34DCKR, U7 74LVC1G17, U8 74LVC2G34DCKR, U9 74LVC2G34DCKR

Commit message: Try to save correct file to repository
"single_buffers" is correct file, NOT  "single_buff"
Parts:
- added C2: 100n, Capacitor_SMD:C_0805_2012Metric_Pad1.18x1.45mm_HandSolder, F.Cu at (259.2, 37.8)
- added C3: 100n, Capacitor_SMD:C_0805_2012Metric_Pad1.18x1.45mm_HandSolder, F.Cu at (259.2, 40.8)
- added C4: 100n, Capacitor_SMD:C_0805_2012Metric_Pad1.18x1.45mm_HandSolder, F.Cu at (259.2, 43.8)
- added C7: 100n, Capacitor_SMD:C_0805_2012Metric_Pad1.18x1.45mm_HandSolder, F.Cu at (259.2, 46.8)
- added C8: 100n, Capacitor_SMD:C_0805_2012Metric_Pad1.18x1.45mm_HandSolder, F.Cu at (259.2, 49.8)
- U1, U12, U13, U14, U15, U16, U17, U18, U19, U2, U3, U4, U5, U6, U8, U9: footprint 74LVC2G34DKCR:74LVC2G34DKCR -> 74LVC2G34DKCR:74LVC2G34DKCR-M
- moved U3 128.8 mm to (98.2, 18.0)
- moved U19 108.8 mm to (188.1, 132.4)
- moved U18 91.6 mm to (207.9, 118.7)
- moved U6 90.7 mm to (149.2, 68.7), turned to 90 degrees
- moved U4 85.9 mm to (267.8, 112.0)
- moved U8 85.3 mm to (154.6, 71.4)
- moved U13 80.7 mm to (208.2, 105.2)
- moved R30 79.4 mm to (213.9, 118.8)
- moved U9 65.1 mm to (275.9, 84.0)
- moved U17 58.2 mm to (208.2, 77.8)
- moved U15 55.8 mm to (250.6, 90.7)
- moved C1 53.6 mm to (195.8, 154.2)
- moved C13 53.6 mm to (195.8, 157.0)
- moved C6 53.6 mm to (195.8, 159.7)
- moved R25 52.1 mm to (212.9, 66.8), turned to -135 degrees
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- renumbered C7 to C1, C5 to C11, C8 to C12, C9 to C13, C4 to C14, C1 to C5, C2 to C6, C6 to C9, JR4 to JR1, JR3 to JR2, JR2 to JR3, JR1 to JR4, R20 to R1, R34 to R16, R30 to R17, R8 to R18, R35 to R19, R33 to R20, R9 to R21, R31 to R22, R10 to R23, R17 to R24, R11 to R25, R32 to R26, R12 to R27, R13 to R28, R14 to R29, R19 to R3, R15 to R30, R16 to R31, R18 to R4, R29 to R5, R5 to R6, R36 to R7
Connections:
- C1 pad 1: unconnected-(C7-Pad1) -> Net-(U10-GPIO15)
- C1 pad 2: unconnected-(C7-Pad2) -> GND
- C10 pad 1: unconnected-(C10-Pad1) -> Net-(U10-GPIO2)
- C10 pad 2: unconnected-(C10-Pad2) -> GND
- C11 pad 1: unconnected-(C5-Pad1) -> Net-(U10-GPIO2)
- C11 pad 2: unconnected-(C5-Pad2) -> GND
- C12 pad 1: unconnected-(C8-Pad1) -> Net-(U10-GPIO1)
- C12 pad 2: unconnected-(C8-Pad2) -> GND
- C13 pad 1: unconnected-(C9-Pad1) -> Net-(U10-GPIO1)
- C13 pad 2: unconnected-(C9-Pad2) -> GND
- C14 pad 1: unconnected-(C4-Pad1) -> GND
- C14 pad 2: unconnected-(C4-Pad2) -> Net-(U10-GPIO1)
- C5 pad 1: unconnected-(C1-Pad1) -> GND
- C5 pad 2: unconnected-(C1-Pad2) -> Net-(U10-GPIO10)
- C6 pad 1: unconnected-(C2-Pad1) -> GND
- C6 pad 2: unconnected-(C2-Pad2) -> 3_3V_Pico
- C9 pad 1: unconnected-(C6-Pad1) -> Net-(U10-GPIO3)
- C9 pad 2: unconnected-(C6-Pad2) -> GND
- J16 pad 1: unconnected-(J16-In-Pad1) -> Net-(J16-In)
- J17 pad 1: unconnected-(J17-In-Pad1) -> Net-(J17-In)
- JR1 pad 1: unconnected-(JR4-Pad1) -> GND
- JR1 pad 2: unconnected-(JR4-Pad2) -> GND
- JR2 pad 1: unconnected-(JR3-Pad1) -> GND
- JR2 pad 2: unconnected-(JR3-Pad2) -> GND
- JR3 pad 1: unconnected-(JR2-Pad1) -> GND
- JR3 pad 2: unconnected-(JR2-Pad2) -> GND
- JR4 pad 1: unconnected-(JR1-Pad1) -> GND
- JR4 pad 2: unconnected-(JR1-Pad2) -> GND
- JR5 pad 1: unconnected-(JR5-Pad1) -> GND
- JR5 pad 2: unconnected-(JR5-Pad2) -> GND
- R1 pad 1: unconnected-(R20-Pad1) -> Net-(U10-GPIO15)
- R1 pad 2: unconnected-(R20-Pad2) -> GND
- R16 pad 1: unconnected-(R34-Pad1) -> GND
- R16 pad 2: unconnected-(R34-Pad2) -> Net-(J16-In)
- R17 pad 1: unconnected-(R30-Pad1) -> GND
- R17 pad 2: unconnected-(R30-Pad2) -> Net-(U10-GPIO9)
- R19 pad 1: unconnected-(R35-Pad1) -> Net-(J17-In)
- R19 pad 2: unconnected-(R35-Pad2) -> Net-(R19-Pad2)
- R20 pad 1: unconnected-(R33-Pad1) -> Net-(J17-In)
- R20 pad 2: unconnected-(R33-Pad2) -> GND
- R22 pad 1: unconnected-(R31-Pad1) -> GND
- R22 pad 2: unconnected-(R31-Pad2) -> Net-(U10-GPIO7)
- R24 pad 1: unconnected-(R17-Pad1) -> GND
- R24 pad 2: unconnected-(R17-Pad2) -> Net-(U10-GPIO6)
- R26 pad 1: unconnected-(R32-Pad1) -> Net-(U10-GPIO5)
- R26 pad 2: unconnected-(R32-Pad2) -> GND
- R3 pad 1: unconnected-(R19-Pad1) -> GND
- R3 pad 2: unconnected-(R19-Pad2) -> Net-(U10-GPIO14)
- R4 pad 1: unconnected-(R18-Pad1) -> GND
- R4 pad 2: unconnected-(R18-Pad2) -> Net-(U10-GPIO13)
- R5 pad 1: unconnected-(R29-Pad1) -> GND
- R5 pad 2: unconnected-(R29-Pad2) -> Net-(U10-GPIO11)
- R7 pad 1: unconnected-(R36-Pad1) -> Net-(J16-In)
- R7 pad 2: unconnected-(R36-Pad2) -> Net-(R7-Pad2)
- U1 pad 4: Net-(U1A-1Y) -> do15
- U1 pad 6: Net-(U1A-1Y) -> do15
- U11 pad 2: unconnected-(U11-Pad2) -> Net-(R19-Pad2)
- U11 pad 3: unconnected-(U11-GND-Pad3) -> GND
- U3 pad 4: Net-(U3A-1Y) -> do13
- U3 pad 6: Net-(U3A-1Y) -> do13
- U4 pad 4: Net-(U4A-1Y) -> do11
- U4 pad 6: Net-(U4A-1Y) -> do11
- U6 pad 4: Net-(U6A-1Y) -> do10
- U6 pad 6: Net-(U6A-1Y) -> do10
- U7 pad 2: unconnected-(U7-Pad2) -> Net-(R7-Pad2)
- U7 pad 3: unconnected-(U7-GND-Pad3) -> GND
- U8 pad 4: Net-(U8A-1Y) -> do9
- U8 pad 6: Net-(U8A-1Y) -> do9
Routing:
- net (no net): track 39.8 -> 750.6 mm
- net Net-(IC3-B0): track 78.4 -> 0.00 mm
- net Net-(IC3-B2): track 75.7 -> 0.00 mm
- net Net-(IC3-B4): track 72.6 -> 0.00 mm
- net Net-(IC3-B6): track 70.5 -> 0.00 mm
- net Net-(IC4-B2): track 61.7 -> 0.00 mm
- net Net-(IC4-B0): track 61.7 -> 0.00 mm
- net Net-(IC4-B6): track 61.2 -> 0.00 mm
- net Net-(IC4-B4): track 60.7 -> 0.00 mm
- net Net-(IC2-B0): track 56.7 -> 0.00 mm
- net Net-(IC2-B2): track 51.9 -> 0.00 mm
- net 3_3V_Pico: track 279.5 -> 233.1 mm
- net Net-(IC2-B4): track 44.3 -> 0.00 mm
- net Net-(IC2-B6): track 39.7 -> 0.00 mm
- net Net-(IC1-B0): track 37.9 -> 0.00 mm
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