File: KiCAD/PrawnDO_Breakout_Connectorized_single_buffers.kicad_sch (KiCad schematic)
At the start: 89 parts, among them J1 do15, J10 do6, J11 do5, J12 do4, J13 do3, J14 do2, J15 do1, J16 Ext. Trig., J17 Ext. Clk., J18 do0, J2 do14, J3 do13, J4 do11, J5 do12, J6 do10, J7 do9, J8 do8, J9 do7, U1 74LVC2G34DCKR, U10 Pico, U11 74LVC1G34, U12 74LVC2G34DCKR, U13 74LVC2G34DCKR, U14 74LVC2G34DCKR, U15 74LVC2G34DCKR, U16 74LVC2G34DCKR, U17 74LVC2G34DCKR, U18 74LVC2G34DCKR, U19 74LVC2G34DCKR, U2 74LVC2G34DCKR, U3 74LVC2G34DCKR, U4 74LVC2G34DCKR, U5 74LVC2G34DCKR, U6 74LVC2G34DCKR, U7 74LVC1G17, U8 74LVC2G34DCKR, U9 74LVC2G34DCKR

Commit message: Try to save correct file to repository
"single_buffers" is correct file, NOT  "single_buff"
Parts:
- removed R1, R3, R4, R6, R7: 49.9, Resistor_SMD:R_1206_3216Metric_Pad1.30x1.75mm_HandSolder, symbol Device:R
- removed R21, R22, R23, R24, R25, R26, R27, R28: 10k, Resistor_SMD:R_0805_2012Metric_Pad1.20x1.40mm_HandSolder, symbol Device:R
- added C2, C4, C7, C8: 100n, Capacitor_SMD:C_0805_2012Metric_Pad1.18x1.45mm_HandSolder, symbol Device:C
- U1, U12, U13, U14, U15, U16, U17, U18, U19, U2, U3, U4, U5, U6, U8, U9: footprint 74LVC2G34DKCR:74LVC2G34DKCR -> 74LVC2G34DKCR:74LVC2G34DKCR-M
- renumbered C7 to C1, C5 to C11, C8 to C12, C9 to C13, C4 to C14, C1 to C5, C2 to C6, C6 to C9, JR4 to JR1, JR3 to JR2, JR2 to JR3, JR1 to JR4, R20 to R1, R34 to R16, R30 to R17, R8 to R18, R35 to R19, R33 to R20, R9 to R21, R31 to R22, R10 to R23, R17 to R24, R11 to R25, R32 to R26, R12 to R27, R13 to R28, R14 to R29, R19 to R3, R15 to R30, R16 to R31, R18 to R4, R29 to R5, R5 to R6, R36 to R7
Connections:
- net 3_3V_Pico: now also C1.1, C10.1, C11.1, C12.1, C13.1, C14.2, C3.1, C5.2, C6.2, C9.1, C2.1, C7.1, C8.1
- net GND: now also C1.2, C10.2, C11.2, C12.2, C13.2, C14.1, C3.2, C5.1, C6.1, C9.2, JR1.1, JR1.2, JR2.1, JR2.2, JR3.1, JR3.2, JR4.1, JR4.2, JR5.1, JR5.2, R1.2, R16.1, R17.1, R20.2, R22.1, R24.1, R26.2, R3.1, R4.1, R5.1, U10.23 (GND), U10.28 (GND), U10.38 (GND), U10.42 (GND), U11.3 (GND), U7.3 (GND), C2.2, C4.2, C7.2, C8.2
- net do10: now also U6.4 (2Y), U6.6 (1Y)
- net do11: now also U4.4 (2Y), U4.6 (1Y)
- net do13: now also U3.4 (2Y), U3.6 (1Y)
- net do15: now also U1.4 (2Y), U1.6 (1Y)
- net do9: now also U8.4 (2Y), U8.6 (1Y)
- net at J17.1 (In): now also R19.1, R20.1
- net at R7.1: now also J16.1 (In), R16.2
- net at R7.2: now also U7.2
- net at U10.17 (GPIO13), U3.1 (1A), U3.3 (2A): now also R4.2
- net at U10.10 (GPIO7), U10.11 (GPIO8), U12.1 (1A)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: now also R22.2
- net at U1.1 (1A), U1.3 (2A), U10.20 (GPIO15): now also R1.1
- net at R26.1: now also U10.7 (GPIO5), U14.1 (1A), U14.3 (2A)
- net at U10.12 (GPIO9), U8.1 (1A), U8.3 (2A): now also R17.2
- net at U10.19 (GPIO14), U2.1 (1A), U2.3 (2A): now also R3.2
- net at R24.2: now also U10.9 (GPIO6), U13.1 (1A), U13.3 (2A)
- net at U10.15 (GPIO11), U4.1 (1A), U4.3 (2A): now also R5.2
- net at R19.2: now also U11.2
Other:
- moved on the sheet: C1, C10, C11, C12, C13, C14, C5, C6, C9, JR1, JR2, JR3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
