File: KiCAD/single buffers/staggered/PrawnDO_Breakout_Connectorized_single_buffers_staggered.kicad_sch (KiCad schematic)
At the start: 80 parts, among them J1 do15, J10 do6, J11 do5, J12 do4, J13 do3, J14 do2, J15 do1, J16 Ext. Trig., J17 Ext. Clk., J18 do0, J2 do14, J3 do13, J4 do11, J5 do12, J6 do10, J7 do9, J8 do8, J9 do7, U1 74LVC2G34DCKR, U10 Pico, U11 74LVC1G34, U12 74LVC2G34DCKR, U13 74LVC2G34DCKR, U14 74LVC2G34DCKR, U15 74LVC2G34DCKR, U16 74LVC2G34DCKR, U17 74LVC2G34DCKR, U18 74LVC2G34DCKR, U19 74LVC2G34DCKR, U2 74LVC2G34DCKR, U3 74LVC2G34DCKR, U4 74LVC2G34DCKR, U5 74LVC2G34DCKR, U6 74LVC2G34DCKR, U7 74LVC1G17, U8 74LVC2G34DCKR, U9 74LVC2G34DCKR

Commit message: Lots of changes
Reorganized the way the different iterations are separated

made double element single buffer (DESB)file, a DESB staggered, and a regular file with the vertically mounted SMAs

made various changes to schematics
Parts:
- added JR10, JR11, JR7, JR8, JR9: 0, Resistor_SMD:R_2010_5025Metric_Pad1.40x2.65mm_HandSolder, symbol Device:R
- added R24, R25, R26, R27, R28: 49.9, Resistor_SMD:R_1206_3216Metric_Pad1.30x1.75mm_HandSolder, symbol Device:R
- added U20, U21: 74LVC1G34, Package_TO_SOT_SMD:SOT-23-5_HandSoldering, symbol 74xGxx:74LVC1G34
- U1, U12, U13, U14, U15, U16, U17, U18, U19, U2, U3, U4, U5, U6, U8, U9: footprint 74LVC2G34DKCR:74LVC2G34DKCR-M -> Package_TO_SOT_SMD:SOT-23-6_Handsoldering
- U10: footprint RPi_Pico:RPi_Pico_SMD_TH -> MCU_RaspberryPi_and_Boards:RPi_Pico_SMD
- renumbered C3 to C1, C5 to C10, C4 to C11, C6 to C2, C8 to C3, C9 to C4, C1 to C5, C2 to C6, C10 to C7, C11 to C8, C7 to C9, JR5 to JR1, JR4 to JR2, JR2 to JR4, JR1 to JR5, R18 to R10, R16 to R11, R19 to R12, R21 to R13, R22 to R14, R23 to R15, R24 to R16, R25 to R17, R26 to R18, R27 to R19, R28 to R20, R29 to R21, R30 to R22, R31 to R23, R20 to R7, R7 to R8, R17 to R9
Connections:
- net 3_3V_Pico: now also C11.1, U21.5 (VCC)
- net GND: now also J10.2 (Ext), J11.2 (Ext), JP1.1 (A), R12.1, R8.1, U10.33 (AGND), JR10.1, JR10.2, JR11.1, JR11.2, JR7.1, JR7.2, JR8.1, JR8.2, JR9.1, JR9.2, U21.3 (GND); no longer R11.1, R7.2
- net do10: now also R27.2; no longer U6.4 (2Y), U6.6 (1Y)
- net do11: now also R26.2; no longer U4.4 (2Y), U4.6 (1Y)
- net do13: now also R25.2; no longer U3.4 (2Y), U3.6 (1Y)
- net do15: now also R24.2; no longer U1.4 (2Y), U1.6 (1Y)
- net do6: now also R15.1; no longer R15.2
- net do9: now also R28.2; no longer U8.4 (2Y), U8.6 (1Y)
- net at R8.2: now also J16.1 (In), R7.1; no longer U7.2
- net at R4.2, U10.17 (GPIO13), U3.3 (2A): now also U5.1 (1A); no longer U3.1 (1A)
- net at R6.1, U5.4 (2Y): now also U21.4; no longer U5.6 (1Y)
- net at R14.2, U10.10 (GPIO7), U12.1 (1A)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: no longer U10.11 (GPIO8), U9.1 (1A), U9.3 (2A)
- net at R13.1, U12.4 (2Y): now also U12.6 (1Y)
- net at R1.1, U1.3 (2A), U10.20 (GPIO15): now also U2.1 (1A); no longer U1.1 (1A)
- net at U10.16 (GPIO12), U5.3 (2A): now also U21.2; no longer U5.1 (1A)
- net at R3.2, U10.19 (GPIO14), U2.3 (2A): now also U3.1 (1A); no longer U2.1 (1A)
- net at R2.1, U2.4 (2Y): now also U3.6 (1Y); no longer U2.6 (1Y)
- net at U13.4 (2Y), U13.6 (1Y): now also R15.2; no longer R15.1
- net at R12.2: now also J17.1 (In), R11.2; no longer U11.2
- new net: R25.1, U3.4 (2Y), U5.6 (1Y)
- new net: R7.2, U7.2
- new net: R24.1, U1.4 (2Y), U2.6 (1Y)
- new net: U10.11 (GPIO8), U9.1 (1A), U9.3 (2A)
- new net: R28.1, U8.4 (2Y), U8.6 (1Y)
- new net: R11.1, U11.2
- new net: R26.1, U4.4 (2Y), U4.6 (1Y)
- new net: R27.1, U6.4 (2Y), U6.6 (1Y)
Other:
- moved on the sheet: J1, J2, J3, J5, JR1, JR2, JR3, JR4, JR5, R1, R11, R12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
