File: KiCAD/major changes/SMA in board/PrawnDO_Breakout_Connectorized_sma_in_board.kicad_sch (KiCad schematic)
At the start: 65 parts, among them IC1 74LVT245D,118, IC2 74LVT245D,118, IC3 74LVT245D,118, IC4 74LVT245D,118, J1 do15, J10 do6, J11 do5, J12 do4, J13 do3, J14 do2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

Commit message: Moved components to be spaced more nicely and shrunk overall size of board
Next is adding holes to connect the prawnblaster
Parts:
- removed C1: 100n, Capacitor_SMD:C_0805_2012Metric_Pad1.18x1.45mm_HandSolder, symbol Device:C
- J1, J10, J11, J12, J13, J14, J15, J16, J2, J3, J4, J5, J6, J7, J8, J9: footprint Connector_Coaxial:SMA_Amphenol_132134_Vertical -> Connector_Coaxial:SMA_Amphenol_901-144_Vertical
Connections:
- net GND: now also J10.2 (Ext), J11.2 (Ext), J12.2 (Ext), J9.2 (Ext)

Commit message: Moved components, added headers, changed transmission track widths, moved mounting hole placement
Changed Capacitor footprints from 0806 to 1210
Parts:
- added H1, H2, H3, H4: MountingHole, MountingHole:MountingHole_3.2mm_M3_ISO7380, symbol Mechanical:MountingHole
- added J19: Conn_01x03, Connector_Molex:Molex_SL_171971-0003_1x03_P2.54mm_Vertical, symbol Connector_Generic:Conn_01x03
- added J20: Conn_01x02, Connector_Molex:Molex_SL_171971-0002_1x02_P2.54mm_Vertical, symbol Connector_Generic:Conn_01x02
- C2, C3: footprint Capacitor_SMD:C_0805_2012Metric_Pad1.18x1.45mm_HandSolder -> Capacitor_SMD:C_1210_3225Metric_Pad1.33x2.70mm_HandSolder
Connections:
- net 3_3V_Pico: now also J19.1 (Pin_1)
- net GND: now also J20.1 (Pin_1)
- new net Ext. Power: J19.3 (Pin_3), J20.2 (Pin_2)
- new net Power  Supply: J19.2 (Pin_2)
Changed lines of the file:
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@@
   (junction (at 226.06 104.14) (diameter 0) (color 0 0 0 0)
   )
-  (junction (at 60.96 46.99) (diameter 0) (color 0 0 0 0)
-  )
   (junction (at 172.72 93.98) (diameter 0) (color 0 0 0 0)
   )
@@
     (stroke (width 0) (type default))
   )
-  (wire (pts (xy 60.96 46.99) (xy 60.96 57.15))
+  (wire (pts (xy 60.96 43.18) (xy 60.96 57.15))
     (stroke (width 0) (type default))
   )
@@
     (stroke (width 0) (type default))
   )
-  (wire (pts (xy 77.47 46.99) (xy 60.96 46.99))
-    (stroke (width 0) (type default))
-  )
   (wire (pts (xy 186.055 122.555) (xy 184.785 122.555))
     (stroke (width 0) (type default))
@@
     (stroke (width 0) (type default))
   )
+  (wire (pts (xy 58.42 31.75) (xy 58.42 43.18))
+    (stroke (width 0) (type default))
+  )
   (wire (pts (xy 181.61 99.06) (xy 187.325 99.06))
     (stroke (width 0) (type default))
@@
     (stroke (width 0) (type default))
   )
-  (wire (pts (xy 60.96 43.18) (xy 60.96 46.99))
-    (stroke (width 0) (type default))
-  )
   (wire (pts (xy 175.895 104.14) (xy 187.325 104.14))
     (stroke (width 0) (type default))
@@
     (stroke (width 0) (type default))
   )
+  (wire (pts (xy 45.085 43.18) (xy 55.88 43.18))
+    (stroke (width 0) (type default))
+  )
   (wire (pts (xy 137.795 34.29) (xy 137.795 67.31))
     (stroke (width 0) (type default))
@@
     )
   )
+  (global_label "Power  Supply" (shape input) (at 58.42 31.75 0) (fields_autoplaced)
+    (effects (font (size 1.27 1.27)) (justify left))
+    (property "Intersheetrefs" "${INTERSHEET_REFS}" (at 75.254 31.75 0)
+      (effects (font (size 1.27 1.27)) (justify left) hide)
+    )
+  )
+  (global_label "Ext. Power" (shape input) (at 48.26 43.18 90) (fields_autoplaced)
+    (effects (font (size 1.27 1.27)) (justify left))
+    (property "Intersheetrefs" "${INTERSHEET_REFS}" (at 48.26 30.0953 90)
+      (effects (font (size 1.27 1.27)) (justify left) hide)
+    )
+  )
   (global_label "3_3V_Pico" (shape input) (at 86.36 107.95 0) (fields_autoplaced)
     (effects (font (size 1.27 1.27)) (justify left))
@@
     )
   )
+  (symbol (lib_id "Connector_Generic:Conn_01x03") (at 58.42 38.1 270) (mirror x) (unit 1)
+    (in_bom yes) (on_board yes) (dnp no)
+    (property "Reference" "J19" (at 53.34 36.83 90)
+      (effects (font (size 1.27 1.27)) (justify right))
+    )
+    (property "Value" "Conn_01x03" (at 53.34 39.37 90)
+      (effects (font (size 1.27 1.27)) (justify right))
+    )
+    (property "Footprint" "Connector_Molex:Molex_SL_171971-0003_1x03_P2.54mm_Vertical" (at 58.42 38.1 0)
+      (effects (font (size 1.27 1.27)) hide)
+    )
+    (property "Datasheet" "~" (at 58.42 38.1 0)
+      (effects (font (size 1.27 1.27)) hide)
+    )
+    (pin "3")
+    (pin "2")
+    (pin "1")
+    (instances
+      (project "PrawnDO_Breakout_Connectorized_sma_in_board"
+        (path "/afe7a1c5-73e2-42c7-95cc-d8f50de6e194"
+          (reference "J19") (unit 1)
+        )
+      )
+    )
+  )
   (symbol (lib_id "Connector:Conn_Coaxial") (at 276.225 74.93 0) (unit 1)
     (in_bom yes) (on_board yes) (dnp no) (fields_autoplaced)
@@
     )
   )
+  (symbol (lib_id "Mechanical:MountingHole") (at 271.145 161.29 0) (unit 1)
+    (in_bom yes) (on_board yes) (dnp no) (fields_autoplaced)
+    (property "Reference" "H4" (at 273.685 160.02 0)
+      (effects (font (size 1.27 1.27)) (justify left))
+    )
+    (property "Value" "MountingHole" (at 273.685 162.56 0)
+      (effects (font (size 1.27 1.27)) (justify left))
+    )
+    (property "Footprint" "MountingHole:MountingHole_3.2mm_M3_ISO7380" (at 271.145 161.29 0)
+      (effects (font (size 1.27 1.27)) hide)
+    )
+    (property "Datasheet" "~" (at 271.145 161.29 0)
+      (effects (font (size 1.27 1.27)) hide)
+    )
+    (instances
+      (project "PrawnDO_Breakout_Connectorized_sma_in_board"
+        (path "/afe7a1c5-73e2-42c7-95cc-d8f50de6e194"
+          (reference "H4") (unit 1)
+        )
+      )
+    )
+  )
   (symbol (lib_id "Device:C") (at 67.31 57.15 90) (unit 1)
     (in_bom yes) (on_board yes) (dnp no) (fields_autoplaced)
@@
       (effects (font (size 1.27 1.27)))
     )
-    (property "Footprint" "Capacitor_SMD:C_0805_2012Metric_Pad1.18x1.45mm_HandSolder" (at 71.12 56.1848 0)
+    (property "Footprint" "Capacitor_SMD:C_1210_3225Metric_Pad1.33x2.70mm_HandSolder" (at 71.12 56.1848 0)
       (effects (font (size 1.27 1.27)) hide)
     )
@@
     )
   )
+  (symbol (lib_id "Mechanical:MountingHole") (at 251.46 149.225 0) (unit 1)
+    (in_bom yes) (on_board yes) (dnp no) (fields_autoplaced)
+    (property "Reference" "H1" (at 254 147.955 0)
+      (effects (font (size 1.27 1.27)) (justify left))
+    )
+    (property "Value" "MountingHole" (at 254 150.495 0)
+      (effects (font (size 1.27 1.27)) (justify left))
+    )
+    (property "Footprint" "MountingHole:MountingHole_3.2mm_M3_ISO7380" (at 251.46 149.225 0)
+      (effects (font (size 1.27 1.27)) hide)
+    )
+    (property "Datasheet" "~" (at 251.46 149.225 0)
+      (effects (font (size 1.27 1.27)) hide)
+    )
+    (instances
+      (project "PrawnDO_Breakout_Connectorized_sma_in_board"
+        (path "/afe7a1c5-73e2-42c7-95cc-d8f50de6e194"
+          (reference "H1") (unit 1)
+        )
+      )
+    )
+  )
   (symbol (lib_id "power:GND") (at 151.765 41.275 270) (unit 1)
     (in_bom yes) (on_board yes) (dnp no) (fields_autoplaced)
@@
     )
   )
+  (symbol (lib_id "power:GND") (at 42.545 43.18 180) (unit 1)
+    (in_bom yes) (on_board yes) (dnp no) (fields_autoplaced)
+    (property "Reference" "#PWR05" (at 42.545 36.83 0)
+      (effects (font (size 1.27 1.27)) hide)
+    )
+    (property "Value" "GND" (at 42.545 38.1 0)
+      (effects (font (size 1.27 1.27)))
+    )
+    (property "Footprint" "" (at 42.545 43.18 0)
+      (effects (font (size 1.27 1.27)) hide)
+    )
+    (property "Datasheet" "" (at 42.545 43.18 0)
+      (effects (font (size 1.27 1.27)) hide)
+    )
+    (pin "1")
+    (instances
+      (project "PrawnDO_Breakout_Connectorized_sma_in_board"
+        (path "/afe7a1c5-73e2-42c7-95cc-d8f50de6e194"
+          (reference "#PWR05") (unit 1)
+        )
+      )
+    )
+  )
   (symbol (lib_id "Device:R") (at 147.955 121.285 0) (unit 1)
     (in_bom yes) (on_board yes) (dnp no)
@@
     )
   )
+  (symbol (lib_id "Mechanical:MountingHole") (at 251.46 161.29 0) (unit 1)
+    (in_bom yes) (on_board yes) (dnp no) (fields_autoplaced)
+    (property "Reference" "H3" (at 254 160.02 0)
+      (effects (font (size 1.27 1.27)) (justify left))
+    )
+    (property "Value" "MountingHole" (at 254 162.56 0)
+      (effects (font (size 1.27 1.27)) (justify left))
+    )
+    (property "Footprint" "MountingHole:MountingHole_3.2mm_M3_ISO7380" (at 251.46 161.29 0)
+      (effects (font (size 1.27 1.27)) hide)
+    )
+    (property "Datasheet" "~" (at 251.46 161.29 0)
+      (effects (font (size 1.27 1.27)) hide)
+    )
+    (instances
+      (project "PrawnDO_Breakout_Connectorized_sma_in_board"
+        (path "/afe7a1c5-73e2-42c7-95cc-d8f50de6e194"
+          (reference "H3") (unit 1)
+        )
+      )
+    )
+  )
   (symbol (lib_id "Device:R") (at 177.8 95.885 270) (unit 1)
     (in_bom yes) (on_board yes) (dnp no)
@@
     )
   )
+  (symbol (lib_id "Connector_Generic:Conn_01x02") (at 42.545 48.26 90) (mirror x) (unit 1)
+    (in_bom yes) (on_board yes) (dnp no) (fields_autoplaced)
+    (property "Reference" "J20" (at 48.26 46.99 90)
+      (effects (font (size 1.27 1.27)) (justify right))
+    )
+    (property "Value" "Conn_01x02" (at 48.26 49.53 90)
+      (effects (font (size 1.27 1.27)) (justify right))
+    )
+    (property "Footprint" "Connector_Molex:Molex_SL_171971-0002_1x02_P2.54mm_Vertical" (at 42.545 48.26 0)
+      (effects (font (size 1.27 1.27)) hide)
+    )
+    (property "Datasheet" "~" (at 42.545 48.26 0)
+      (effects (font (size 1.27 1.27)) hide)
+    )
+    (pin "1")
+    (pin "2")
+    (instances
+      (project "PrawnDO_Breakout_Connectorized_sma_in_board"
+        (path "/afe7a1c5-73e2-42c7-95cc-d8f50de6e194"
+          (reference "J20") (unit 1)
+        )
+      )
+    )
+  )
   (symbol (lib_id "Device:R") (at 192.405 66.675 270) (unit 1)
     (in_bom yes) (on_board yes) (dnp no)
@@
     )
   )
+  (symbol (lib_id "Mechanical:MountingHole") (at 271.145 149.225 0) (unit 1)
+    (in_bom yes) (on_board yes) (dnp no) (fields_autoplaced)
+    (property "Reference" "H2" (at 273.685 147.955 0)
+      (effects (font (size 1.27 1.27)) (justify left))
+    )
+    (property "Value" "MountingHole" (at 273.685 150.495 0)
+      (effects (font (size 1.27 1.27)) (justify left))
+    )
+    (property "Footprint" "MountingHole:MountingHole_3.2mm_M3_ISO7380" (at 271.145 149.225 0)
+      (effects (font (size 1.27 1.27)) hide)
+    )
+    (property "Datasheet" "~" (at 271.145 149.225 0)
+      (effects (font (size 1.27 1.27)) hide)
+    )
+    (instances
+      (project "PrawnDO_Breakout_Connectorized_sma_in_board"
+        (path "/afe7a1c5-73e2-42c7-95cc-d8f50de6e194"
+          (reference "H2") (unit 1)
+        )
+      )
+    )
+  )
   (symbol (lib_id "Device:R") (at 219.075 104.14 90) (unit 1)
     (in_bom yes) (on_board yes) (dnp no)
@@
       (effects (font (size 1.27 1.27)))
     )
-    (property "Footprint" "Capacitor_SMD:C_0805_2012Metric_Pad1.18x1.45mm_HandSolder" (at 72.39 84.1248 0)
+    (property "Footprint" "Capacitor_SMD:C_1210_3225Metric_Pad1.33x2.70mm_HandSolder" (at 72.39 84.1248 0)
       (effects (font (size 1.27 1.27)) hide)
     )

Commit message: Trace changes
Fixed some traces and added a connection to ground through pins on pico

Also made slot for USB slightly larger.

Moved resistor on bottom of board

Changed header footprint
Parts:
- C2, C3: footprint Capacitor_SMD:C_1210_3225Metric_Pad1.33x2.70mm_HandSolder -> Capacitor_SMD:C_1206_3216Metric_Pad1.33x1.80mm_HandSolder
- J19: value Conn_01x03 -> PWR SEL; footprint Connector_Molex:Molex_SL_171971-0003_1x03_P2.54mm_Vertical -> Connector_PinHeader_2.54mm:PinHeader_1x03_P2.54mm_Vertical
- J20: value Conn_01x02 -> EXT PWR
Changed lines of the file:
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@@
       (effects (font (size 1.27 1.27)) (justify right))
     )
-    (property "Value" "Conn_01x03" (at 53.34 39.37 90)
-      (effects (font (size 1.27 1.27)) (justify right))
-    )
-    (property "Footprint" "Connector_Molex:Molex_SL_171971-0003_1x03_P2.54mm_Vertical" (at 58.42 38.1 0)
+    (property "Value" "PWR SEL" (at 53.34 39.37 90)
+      (effects (font (size 1.27 1.27)) (justify right))
+    )
+    (property "Footprint" "Connector_PinHeader_2.54mm:PinHeader_1x03_P2.54mm_Vertical" (at 58.42 38.1 0)
       (effects (font (size 1.27 1.27)) hide)
     )
@@
       (effects (font (size 1.27 1.27)) hide)
     )
+    (pin "1")
+    (pin "2")
     (pin "3")
-    (pin "2")
-    (pin "1")
     (instances
       (project "PrawnDO_Breakout_Connectorized_sma_in_board"
@@
       (effects (font (size 1.27 1.27)))
     )
-    (property "Footprint" "Capacitor_SMD:C_1210_3225Metric_Pad1.33x2.70mm_HandSolder" (at 71.12 56.1848 0)
+    (property "Footprint" "Capacitor_SMD:C_1206_3216Metric_Pad1.33x1.80mm_HandSolder" (at 71.12 56.1848 0)
       (effects (font (size 1.27 1.27)) hide)
     )
@@
       (effects (font (size 1.27 1.27)) (justify right))
     )
-    (property "Value" "Conn_01x02" (at 48.26 49.53 90)
+    (property "Value" "EXT PWR" (at 48.26 49.53 90)
       (effects (font (size 1.27 1.27)) (justify right))
     )
@@
       (effects (font (size 1.27 1.27)))
     )
-    (property "Footprint" "Capacitor_SMD:C_1210_3225Metric_Pad1.33x2.70mm_HandSolder" (at 72.39 84.1248 0)
-      (effects (font (size 1.27 1.27)) hide)
-    )
+    (property "Footprint" "Capacitor_SMD:C_1206_3216Metric_Pad1.33x1.80mm_HandSolder" (at 72.39 84.1248 0)
+      (effects (font (size 1.27 1.27)) hide)
+    )

Commit message: Added Hierarchy sheet for mounting holes
ddd
Parts:
- removed H1, H2, H3, H4: MountingHole, MountingHole:MountingHole_3.2mm_M3_ISO7380, symbol Mechanical:MountingHole
Other:
- added sheet Mounts (SMA_in_board_mounts.kicad_sch)
Changed lines of the file:
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@@
-    )
-  )
-  (symbol (lib_id "Mechanical:MountingHole") (at 271.145 161.29 0) (unit 1)
-    (in_bom yes) (on_board yes) (dnp no) (fields_autoplaced)
-    (property "Reference" "H4" (at 273.685 160.02 0)
-      (effects (font (size 1.27 1.27)) (justify left))
-    )
-    (property "Value" "MountingHole" (at 273.685 162.56 0)
-      (effects (font (size 1.27 1.27)) (justify left))
-    )
-    (property "Footprint" "MountingHole:MountingHole_3.2mm_M3_ISO7380" (at 271.145 161.29 0)
-      (effects (font (size 1.27 1.27)) hide)
-    )
-    (property "Datasheet" "~" (at 271.145 161.29 0)
-      (effects (font (size 1.27 1.27)) hide)
-    )
-    (instances
-      (project "PrawnDO_Breakout_Connectorized_sma_in_board"
-        (path "/afe7a1c5-73e2-42c7-95cc-d8f50de6e194"
-          (reference "H4") (unit 1)
-        )
-      )
     )
   )
@@
     )
   )
-  (symbol (lib_id "Mechanical:MountingHole") (at 251.46 149.225 0) (unit 1)
-    (in_bom yes) (on_board yes) (dnp no) (fields_autoplaced)
-    (property "Reference" "H1" (at 254 147.955 0)
-      (effects (font (size 1.27 1.27)) (justify left))
-    )
-    (property "Value" "MountingHole" (at 254 150.495 0)
-      (effects (font (size 1.27 1.27)) (justify left))
-    )
-    (property "Footprint" "MountingHole:MountingHole_3.2mm_M3_ISO7380" (at 251.46 149.225 0)
-      (effects (font (size 1.27 1.27)) hide)
-    )
-    (property "Datasheet" "~" (at 251.46 149.225 0)
-      (effects (font (size 1.27 1.27)) hide)
-    )
-    (instances
-      (project "PrawnDO_Breakout_Connectorized_sma_in_board"
-        (path "/afe7a1c5-73e2-42c7-95cc-d8f50de6e194"
-          (reference "H1") (unit 1)
-        )
-      )
-    )
-  )
   (symbol (lib_id "power:GND") (at 151.765 41.275 270) (unit 1)
     (in_bom yes) (on_board yes) (dnp no) (fields_autoplaced)
@@
     )
   )
-  (symbol (lib_id "Mechanical:MountingHole") (at 251.46 161.29 0) (unit 1)
-    (in_bom yes) (on_board yes) (dnp no) (fields_autoplaced)
-    (property "Reference" "H3" (at 254 160.02 0)
-      (effects (font (size 1.27 1.27)) (justify left))
-    )
-    (property "Value" "MountingHole" (at 254 162.56 0)
-      (effects (font (size 1.27 1.27)) (justify left))
-    )
-    (property "Footprint" "MountingHole:MountingHole_3.2mm_M3_ISO7380" (at 251.46 161.29 0)
-      (effects (font (size 1.27 1.27)) hide)
-    )
-    (property "Datasheet" "~" (at 251.46 161.29 0)
-      (effects (font (size 1.27 1.27)) hide)
-    )
-    (instances
-      (project "PrawnDO_Breakout_Connectorized_sma_in_board"
-        (path "/afe7a1c5-73e2-42c7-95cc-d8f50de6e194"
-          (reference "H3") (unit 1)
-        )
-      )
-    )
-  )
   (symbol (lib_id "Device:R") (at 177.8 95.885 270) (unit 1)
     (in_bom yes) (on_board yes) (dnp no)
@@
         (path "/afe7a1c5-73e2-42c7-95cc-d8f50de6e194"
           (reference "R11") (unit 1)
-        )
-      )
-    )
-  )
-  (symbol (lib_id "Mechanical:MountingHole") (at 271.145 149.225 0) (unit 1)
-    (in_bom yes) (on_board yes) (dnp no) (fields_autoplaced)
-    (property "Reference" "H2" (at 273.685 147.955 0)
-      (effects (font (size 1.27 1.27)) (justify left))
-    )
-    (property "Value" "MountingHole" (at 273.685 150.495 0)
-      (effects (font (size 1.27 1.27)) (justify left))
-    )
-    (property "Footprint" "MountingHole:MountingHole_3.2mm_M3_ISO7380" (at 271.145 149.225 0)
-      (effects (font (size 1.27 1.27)) hide)
-    )
-    (property "Datasheet" "~" (at 271.145 149.225 0)
-      (effects (font (size 1.27 1.27)) hide)
-    )
-    (instances
-      (project "PrawnDO_Breakout_Connectorized_sma_in_board"
-        (path "/afe7a1c5-73e2-42c7-95cc-d8f50de6e194"
-          (reference "H2") (unit 1)
         )
       )
@@
       )
     )
+  )
+  (sheet (at 90.932 148.209) (size 42.418 26.797) (fields_autoplaced)
+    (stroke (width 0.1524) (type solid))
+    (fill (color 90 255 127 1.0000))
+    (property "Sheetname" "Mounts" (at 90.932 147.4974 0)
+      (effects (font (size 1.27 1.27)) (justify left bottom))
+    )
+    (property "Sheetfile" "SMA_in_board_mounts.kicad_sch" (at 90.932 175.5906 0)
+      (effects (font (size 1.27 1.27)) (justify left top))
+    )
+    (instances
+      (project "PrawnDO_Breakout_Connectorized_sma_in_board"
+        (path "/afe7a1c5-73e2-42c7-95cc-d8f50de6e194" (page "3"))
+      )
+    )
